File: TrabajoPractico_laboratorio1/diseñoPlaca.kicad_pcb (KiCad board)
At the start: 2 copper layers, 9 parts

Commit message: TPLAB1
Parts:
- added REF**: OUT-IN, TerminalBlock:TerminalBlock_bornier-2_P5.08mm, F.Cu at (100.0, 76.0)
- moved RF1 2.88 mm to (156.5, 78.6)
- moved RF2 2.42 mm to (162.6, 78.6)
- moved REF** 0.94 mm to (100.0, 63.5)
- moved RZ2 0.12 mm to (149.9, 78.6)
Routing:
- net (no net): track 454.7 -> 473.9 mm
